File: Hardware/inktime_pcb.brd (EAGLE design)
At the start: 46 x 35 mm, 105 parts, among them IC1 BQ25180YBGR_BQ25180YBGR, IC2 RT6160AWSC_RT6160AWSC, IC3 DRV2605YZFR_DRV2605YZFR, IC4 BMA423_BMA423, J1 KH-TYPE-C-16P_KH-TYPE-C-16P, J2 TC2030-IDC_TC2030-IDC, J3 503480-2400_503480-2400, Q1 ESP32_C6_LIBRARY_6_SI1308EDL-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, Q2 20V/4.2A/52mΩ/1.4W, SW1 2025-10-22_07-23-44_LIBRARY_E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, SW2 2025-10-22_07-23-44_LIBRARY_E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, SW3 2025-10-22_07-23-44_LIBRARY_E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, U1 ESP32_C6_LIBRARY_MAX17048G+T10

Commit message: final version
Parts:
- removed L1: 68u, Inktime Library:MLP2016SR47MT0S1_INDC2016X100N
- removed L3, L5: MLP2016SR47MT0S1_FTC252012SR47MBCA, Inktime Library:MLP2016SR47MT0S1_INDC2016X100N
- removed U$1, U$3, U$6, U$9: 10u, Inktime Library:NORDIC_NRF_3_RESC0201_L
- removed U$10, U$14, U$15, U$18, U$26, U$27, U$30: 4.7u, Inktime Library:NORDIC_NRF_3_RESC0201_L
- removed U$11, U$13, U$2, U$28, U$32: 100n, Inktime Library:NORDIC_NRF_3_RESC0201_L
- removed U$16: 100p, Inktime Library:NORDIC_NRF_3_RESC0201_L
- removed U$17, U$23, U$24, U$25, U$7: N.C., Inktime Library:NORDIC_NRF_3_RESC0201_L
- removed U$19, U$21: 12p, Inktime Library:NORDIC_NRF_3_RESC0201_L
- removed U$29: NORDIC_NRF_4_NRF52840_QF, Inktime Library:NORDIC_NRF_4_AQFN50P700X700X85_HS-74N
- removed U$33, U$34, U$36, U$37, U$38, U$39, U$40, U$41, U$42, U$43: 1u/50V, Inktime Library:NORDIC_NRF_3_RESC0201_L
- removed U$35: 0.1u/50V, Inktime Library:NORDIC_NRF_3_RESC0201_L
- added C11, C17: 10u, Inktime Library:ESP32_C6_LIBRARY_1_ESP32_WROVER_EAGLE-LTSPICE_C0402
- added C12, C13: 22u, Inktime Library:ESP32_C6_LIBRARY_1_ESP32_WROVER_EAGLE-LTSPICE_C0402
- added C14: 1.0u, Inktime Library:ESP32_C6_LIBRARY_1_ESP32_WROVER_EAGLE-LTSPICE_C0402
- added C15: 4.7u, Inktime Library:ESP32_C6_LIBRARY_1_ESP32_WROVER_EAGLE-LTSPICE_C0402
- added C16: 4.7u/25V, Inktime Library:ESP32_C6_LIBRARY_1_ESP32_WROVER_EAGLE-LTSPICE_C0402
- added C18, C19, C34, C35, C36: 4.7u, Inktime Library:NORDIC_NRF_3_RESC0201_L
- added C20, C49: 47n, Inktime Library:NORDIC_NRF_3_RESC0201_L
- added C21, C24, C29, C31, C32: N.C, Inktime Library:NORDIC_NRF_3_RESC0201_L
- added C22, C26, C30, C33: 100n, Inktime Library:NORDIC_NRF_3_RESC0201_L
- added C23: 100p, Inktime Library:NORDIC_NRF_3_RESC0201_L
- added C25: 820p, Inktime Library:NORDIC_NRF_3_RESC0201_L
- added C27, C28: 12p, Inktime Library:NORDIC_NRF_3_RESC0201_L
- added C37: 0.1u, Inktime Library:GRM011R60J152KE01L_2_CAPC0201X13N
- added C38, C39, C40, C41, C42, C43, C44, C45, C46, C47: 1u/50V, Inktime Library:NORDIC_NRF_3_RESC0201_L
- added C48: 0.1u/50V, Inktime Library:NORDIC_NRF_3_RESC0201_L
- C3: value 0.1u -> 100n; device Inktime Library:GRM011R60J152KE01L_2_CAPC0201X13N -> Inktime Library:NORDIC_NRF_3_RESC0201_L
- L4: value MLP2016SR47MT0S1_FTC252012SR47MBCA -> 68u; device Inktime Library:MLP2016SR47MT0S1_INDC2016X100N -> Inktime Library:ESP32_C6_LIBRARY_2_IND_4828-WE-TPC_WRE
- U$20: value 32MHz -> 4.7u; device Inktime Library:NORDIC_NRF_BT-XTAL_2016_N -> Inktime Library:NORDIC_NRF_3_RESC0201_L
- U$22: value 820p N.C. -> 32MHz; device Inktime Library:NORDIC_NRF_3_RESC0201_L -> Inktime Library:NORDIC_NRF_BT-XTAL_2016_N
- U$31: value 100n -> NORDIC_NRF_4_NRF52840_QF; device Inktime Library:NORDIC_NRF_3_RESC0201_L -> Inktime Library:NORDIC_NRF_4_AQFN50P700X700X85_HS-74N
- U$4: value N.C. -> 15n; device Inktime Library:NORDIC_NRF_3_RESC0201_L -> Inktime Library:NORDIC_NRF_2_RESC0402_L
- U$5: value N.C. -> (none); device Inktime Library:NORDIC_NRF_3_RESC0201_L -> Inktime Library:NORDIC_NRF_2_RESC0402_L
- U$8: device Inktime Library:NORDIC_NRF_3_RESC0201_L -> Inktime Library:NORDIC_NRF_2_RESC0402_L
- moved J2 36.1 mm to (15.7, -7.54), turned to 0 degrees
- moved TP1 35.4 mm to (18.7, -14.5), turned to 180 degrees
- moved TP5 35.0 mm to (16.9, -15.8), turned to 180 degrees
- moved L4 34.1 mm to (-17.9, 12.4), turned to 180 degrees
- moved TP4 31.5 mm to (14.4, -16.2), turned to 180 degrees
- moved TP3 30.5 mm to (16.9, -12.8), turned to 180 degrees
- moved SJ1 29.8 mm to (-13.7, 14.9), turned to 270 degrees
- moved TP11 28.8 mm to (-22.1, -12.4)
- moved TP10 28.8 mm to (-22.0, -9.75)
- moved U1 28.0 mm to (-11.2, -10.0)
- moved C10 28.0 mm to (-13.3, -10.2)
- moved R2 27.4 mm to (-11.6, 15.7)
- moved R4 27.4 mm to (-12.3, 15.7)
- moved Q1 27.4 mm to (-11.3, 13.5)
- moved R1 27.3 mm to (-10.4, 15.6)
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- renumbered U$12 to X1
Connections:
- removed net D+: D4.4, U$29.P$AD6
- removed net D-: D4.6, U$29.P$AD4
- removed net N$6: L3.1, L4.2
- new net D_N: D4.6, U$31.P$AD4
- new net D_P: D4.4, U$31.P$AD6
- new net N$3: U$4.1, U$8.2
- net 3V1: now also C35.1, U$31.P$AC5; no longer U$27.2, U$29.P$AC5
- net 3V3: now also C12.1, C13.1, C15.1, C22.1, C26.1, C3.1, C33.1, C36.1, U$31.P$A22, U$31.P$AD14, U$31.P$AD23, U$31.P$B1, U$31.P$W1, U$31.P$Y2; no longer U$11.2, U$14.2, U$26.2, U$28.2, U$29.P$A22, U$29.P$AD14, U$29.P$AD23, U$29.P$B1, U$29.P$W1, U$29.P$Y2, U$31.1, U$32.2, U$8.1, U$9.1
- net ALERT: now also U$31.P$J24; no longer U$29.P$J24
- net ANT: now also C29.1, U$31.P$H23, U$5.1; no longer L5.1, U$23.2, U$29.P$H23
- net DEC1: now also C30.1, U$31.P$C1; no longer U$13.2, U$29.P$C1
- net DEC3: now also C23.1, U$31.P$D23; no longer U$16.2, U$29.P$D23
- net DEC4_6: now also C14.1, C20.1, C24.1, U$31.P$B5, U$31.P$E24; no longer L3.2, U$17.2, U$29.P$B5, U$29.P$E24, U$5.2
- net EPD_3V3: now also C17.1, C48.2, L4.2; no longer L1.1, U$1.1, U$35.1
- net EPD_BUSY: now also U$31.P$AD12; no longer U$29.P$AD12
- net EPD_CS: now also U$31.P$K2; no longer U$29.P$K2
- net EPD_DC: now also U$31.P$AD10; no longer U$29.P$AD10
- net EPD_RST: now also U$31.P$AC11; no longer U$29.P$AC11
- net GND: now also C11.2, C12.2, C13.2, C14.2, C15.2, C17.2, C18.1, C19.1, C20.2, C21.2, C22.2, C23.2, C24.2, C25.2, C26.2, C27.2, C28.2, C29.2, C30.2, C31.2, C32.2, C33.2, C34.2, C35.2, C36.2, C37.1, C38.1, C39.1, C40.1, C41.1, C42.1, C43.1, C44.1, C45.1, C46.1, C47.1, C48.1, C49.2, U$22.2, U$22.4, U$31.P$74, U$31.P$75, U$31.P$76, U$31.P$77, U$31.P$78, U$31.P$79, U$31.P$80, U$31.P$81, U$31.P$82, U$31.P$83, U$31.P$84, U$31.P$85, U$31.P$86, U$31.P$87, U$31.P$88, U$31.P$89, U$31.P$90, U$31.P$B7, U$31.P$F23; no longer U$1.2, U$10.1, U$11.1, U$13.1, U$14.1, U$15.1, U$16.1, U$17.1, U$18.2, U$19.1, U$20.4, U$21.1, U$22.1, U$23.1, U$24.1, U$25.1, U$26.1, U$27.1, U$28.1, U$29.P$74, U$29.P$75, U$29.P$76, U$29.P$77, U$29.P$78, U$29.P$79, U$29.P$80, U$29.P$81, U$29.P$82, U$29.P$83, U$29.P$84, U$29.P$85, U$29.P$86, U$29.P$87, U$29.P$88, U$29.P$89, U$29.P$90, U$29.P$B7, U$29.P$F23, U$3.1, U$30.1, U$31.2, U$32.1, U$33.2, U$34.2, U$35.2, U$36.2, U$37.2, U$38.2, U$39.2, U$4.1, U$40.2, U$41.2, U$42.2, U$43.2, U$5.1, U$6.2, U$7.1, U$8.2, U$9.2
- net HAPTIC_EN: now also U$31.P$U1; no longer U$29.P$U1
- net IMU_INT1: now also U$31.P$N1; no longer U$29.P$N1
- net IMU_INT2: now also U$31.P$P2; no longer U$29.P$P2
- net MOSI: now also U$31.P$B13; no longer U$29.P$B13
- net N$1: now also C18.2, U$31.P$D2; no longer U$10.2, U$29.P$D2
- net N$10: now also C31.1, C32.1, U$5.2; no longer L5.2, U$24.2, U$25.2
- net N$11: now also C21.1, U$31.P$A18; no longer U$29.P$A18, U$7.2
- net N$2: now also C19.2, U$31.P$F2; no longer U$15.2, U$29.P$F2
- net N$20: now also C38.2; no longer U$33.1
- net N$21: now also C39.2; no longer U$34.1
- net N$23: now also C16.1; no longer U$2.1
- net N$25: now also C16.2, L4.1; no longer L1.2, U$2.2
- net N$31: now also C40.2; no longer U$36.1
- net N$32: now also C41.2; no longer U$37.1
- net N$33: now also C42.2; no longer U$38.1
- net N$34: now also C43.2; no longer U$39.1
- net N$36: now also C45.2; no longer U$41.1
- net N$38: now also C47.2; no longer U$43.1
- net N$5: now also U$31.P$B3, U$8.1; no longer L4.1, U$29.P$B3
- net N$8: now also C25.1, U$31.P$N24; no longer U$22.2, U$29.P$N24
- net P0.04: now also U$31.P$J1; no longer U$29.P$J1
- net P0.09: now also U$31.P$L24; no longer U$29.P$L24
- net P0.13: now also U$31.P$AD8; no longer U$29.P$AD8
- net P0.14: now also U$31.P$AC9; no longer U$29.P$AC9
- net P0.19: now also U$31.P$AC15; no longer U$29.P$AC15
- net P0.20: now also U$31.P$AD16; no longer U$29.P$AD16
- net P0.21: now also U$31.P$AC17; no longer U$29.P$AC17
- net P0.22: now also U$31.P$AD18; no longer U$29.P$AD18
- net P0.23: now also U$31.P$AC19; no longer U$29.P$AC19
- net P0.24: now also U$31.P$AD20; no longer U$29.P$AD20
- net P0.25: now also U$31.P$AC21; no longer U$29.P$AC21
- net P0.26: now also U$31.P$G1; no longer U$29.P$G1
- net P0.27: now also U$31.P$H2; no longer U$29.P$H2
- net P0.28: now also U$31.P$B11; no longer U$29.P$B11
- net P0.29: now also U$31.P$A10; no longer U$29.P$A10
- net P0.30: now also U$31.P$B9; no longer U$29.P$B9
- net P0.31: now also U$31.P$A8; no longer U$29.P$A8
- net P1.01: now also U$31.P$Y23; no longer U$29.P$Y23
- net P1.02: now also U$31.P$W24; no longer U$29.P$W24
- net P1.03: now also U$31.P$V23; no longer U$29.P$V23
- net P1.04: now also U$31.P$U24; no longer U$29.P$U24
- net P1.05: now also U$31.P$T23; no longer U$29.P$T23
- net P1.06: now also U$31.P$R24; no longer U$29.P$R24
- net P1.07: now also U$31.P$P23; no longer U$29.P$P23
- net P1.09: now also U$31.P$R1; no longer U$29.P$R1
- net P1.10: now also U$31.P$A20; no longer U$29.P$A20
- net P1.11: now also U$31.P$B19; no longer U$29.P$B19
- net P1.12: now also U$31.P$B17; no longer U$29.P$B17
- net P1.13: now also U$31.P$A16; no longer U$29.P$A16
- net P1.14: now also U$31.P$B15; no longer U$29.P$B15
- net P1.15: now also U$31.P$A14; no longer U$29.P$A14
- net PMIC_INT: now also U$31.P$T2; no longer U$29.P$T2
- net PREVGH: now also C44.2; no longer U$40.1
- net PREVGL: now also C46.2; no longer U$42.1
- net RESET: now also U$31.P$AC13; no longer U$29.P$AC13
- net SCK: now also U$31.P$A12; no longer U$29.P$A12
- net SCL: now also U$31.P$M2; no longer U$29.P$M2
- net SDA: now also U$31.P$L1; no longer U$29.P$L1
- net SWDCLK: now also U$31.P$AA24; no longer U$29.P$AA24
- net SWDIO: now also U$31.P$AC24; no longer U$29.P$AC24
- net SWO: now also U$31.P$AD22; no longer U$29.P$AD22
- net VBUS: now also C34.1, U$20.1, U$31.P$AD2; no longer U$18.1, U$29.P$AD2, U$30.2
- net VREG: now also C11.1, C37.2, C49.1; no longer C3.1, U$3.2, U$6.1
- net XC1: now also C28.1, U$22.1, U$31.P$B24; no longer U$20.1, U$21.2, U$29.P$B24
- net XC2: now also C27.1, U$22.3, U$31.P$A23; no longer U$19.2, U$20.3, U$29.P$A23
Routing:
- net 3V3: track 0.00 -> 179.0 mm, vias 0 -> 21
- net VBAT: track 0.00 -> 93.2 mm, vias 0 -> 5
- net SCL: track 0.00 -> 84.4 mm, vias 0 -> 7
- net SDA: track 0.00 -> 81.9 mm, vias 0 -> 4
- net P1.02: track 0.00 -> 49.6 mm, vias 0 -> 2
- net P0.13: track 0.00 -> 44.9 mm, vias 0 -> 2
- net SWO: track 0.00 -> 38.7 mm, vias 0 -> 2
- net EPD_3V3: track 0.00 -> 38.5 mm, vias 0 -> 3
- net SWDCLK: track 0.00 -> 37.4 mm, vias 0 -> 2
- net VBUS: track 0.00 -> 36.6 mm, vias 0 -> 3
- net SWDIO: track 0.00 -> 31.5 mm, vias 0 -> 2
- net P0.14: track 0.00 -> 31.0 mm, vias 0 -> 2
- net ANT: track 0.00 -> 29.8 mm, vias 0 -> 4
- net HAPTIC_EN: track 0.00 -> 28.7 mm, vias 0 -> 5
- net RESET: track 0.00 -> 25.4 mm, vias 0 -> 2
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- added copper zone on layer 1, net 3V3
- added copper zone on layer 2, net 3V3
- added copper zone on layer 1, net EPD_3V3
- added copper zone on layer 1, net LX1
- added copper zone on layer 1, net LX2
- added copper zone on layer 1, net N$25
- added copper zone on layer 1, net VREG
- added copper zone on layer 2, net VREG
