File: Hardware/inktime_schematic.sch (EAGLE design)
At the start: 105 parts, among them IC1 BQ25180YBGR_BQ25180YBGR, IC2 RT6160AWSC_RT6160AWSC, IC3 DRV2605YZFR_DRV2605YZFR, IC4 BMA423_BMA423, J1 KH-TYPE-C-16P_KH-TYPE-C-16P, J2 TC2030-IDC_TC2030-IDC, J3 503480-2400_503480-2400, Q1 ESP32_C6_LIBRARY_6_SI1308EDL-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, Q2 20V/4.2A/52mΩ/1.4W, SW1 2025-10-22_07-23-44_LIBRARY_E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, SW2 2025-10-22_07-23-44_LIBRARY_E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, SW3 2025-10-22_07-23-44_LIBRARY_E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, U1 ESP32_C6_LIBRARY_MAX17048G+T10

Commit message: final version
Parts:
- removed L1: 68u, Inktime Library:MLP2016SR47MT0S1_FTC252012SR47MBCA
- removed L3, L5: MLP2016SR47MT0S1_FTC252012SR47MBCA, Inktime Library:MLP2016SR47MT0S1_FTC252012SR47MBCA
- removed U$1, U$3, U$6, U$9: 10u, Inktime Library:NORDIC_NRF_3_CAPACITOR_0201_L
- removed U$11, U$13, U$2, U$28, U$32: 100n, Inktime Library:NORDIC_NRF_3_CAPACITOR_0201_L
- removed U$14, U$18, U$26, U$27, U$30: 4.7u, Inktime Library:NORDIC_NRF_3_CAPACITOR_0201_L
- removed U$16: 100p, Inktime Library:NORDIC_NRF_3_CAPACITOR_0201_L
- removed U$17, U$23, U$24, U$25, U$7: N.C., Inktime Library:NORDIC_NRF_3_CAPACITOR_0201_L
- removed U$19, U$21: 12p, Inktime Library:NORDIC_NRF_3_CAPACITOR_0201_L
- removed U$29: NORDIC_NRF_4_NRF52840_QF, Inktime Library:NORDIC_NRF_4_NRF52840_QF
- removed U$33, U$34, U$36, U$37, U$38, U$39, U$40, U$41, U$42, U$43: 1u/50V, Inktime Library:NORDIC_NRF_3_CAPACITOR_0201_L
- removed U$35: 0.1u/50V, Inktime Library:NORDIC_NRF_3_CAPACITOR_0201_L
- added C11, C17: 10u, Inktime Library:ESP32_C6_LIBRARY_1_ESP32_WROVER_EAGLE-LTSPICE_CC0402
- added C12, C13: 22u, Inktime Library:ESP32_C6_LIBRARY_1_ESP32_WROVER_EAGLE-LTSPICE_CC0402
- added C14: 1.0u, Inktime Library:ESP32_C6_LIBRARY_1_ESP32_WROVER_EAGLE-LTSPICE_CC0402
- added C15: 4.7u, Inktime Library:ESP32_C6_LIBRARY_1_ESP32_WROVER_EAGLE-LTSPICE_CC0402
- added C16: 4.7u/25V, Inktime Library:ESP32_C6_LIBRARY_1_ESP32_WROVER_EAGLE-LTSPICE_CC0402
- added C20, C49: 47n, Inktime Library:NORDIC_NRF_3_CAPACITOR_0201_L
- added C21, C24, C29, C31, C32: N.C, Inktime Library:NORDIC_NRF_3_CAPACITOR_0201_L
- added C22, C26, C30, C33: 100n, Inktime Library:NORDIC_NRF_3_CAPACITOR_0201_L
- added C23: 100p, Inktime Library:NORDIC_NRF_3_CAPACITOR_0201_L
- added C25: 820p, Inktime Library:NORDIC_NRF_3_CAPACITOR_0201_L
- added C27, C28: 12p, Inktime Library:NORDIC_NRF_3_CAPACITOR_0201_L
- added C34, C35, C36: 4.7u, Inktime Library:NORDIC_NRF_3_CAPACITOR_0201_L
- added C37: 0.1u, Inktime Library:GRM011R60J152KE01L_2_GRM011R60J152KE01L
- added C38, C39, C40, C41, C42, C43, C44, C45, C46, C47: 1u/50V, Inktime Library:NORDIC_NRF_3_CAPACITOR_0201_L
- added C48: 0.1u/50V, Inktime Library:NORDIC_NRF_3_CAPACITOR_0201_L
- C3: value 0.1u -> 100n; device Inktime Library:GRM011R60J152KE01L_2_GRM011R60J152KE01L -> Inktime Library:NORDIC_NRF_3_CAPACITOR_0201_L
- L4: value MLP2016SR47MT0S1_FTC252012SR47MBCA -> 68u; device Inktime Library:MLP2016SR47MT0S1_FTC252012SR47MBCA -> Inktime Library:ESP32_C6_LIBRARY_2_744043680IND_4828-WE-TPC_WRE
- U$20: value 32MHz -> 4.7u; device Inktime Library:NORDIC_NRF_XTAL_32MHZ -> Inktime Library:NORDIC_NRF_3_CAPACITOR_0201_L
- U$22: value 820p N.C. -> 32MHz; device Inktime Library:NORDIC_NRF_3_CAPACITOR_0201_L -> Inktime Library:NORDIC_NRF_XTAL_32MHZ
- U$31: value 100n -> NORDIC_NRF_4_NRF52840_QF; device Inktime Library:NORDIC_NRF_3_CAPACITOR_0201_L -> Inktime Library:NORDIC_NRF_4_NRF52840_QF
- U$4: value N.C. -> 15n; device Inktime Library:NORDIC_NRF_3_CAPACITOR_0201_L -> Inktime Library:NORDIC_NRF_2_INDUCTOR_0402_L
- U$5: value N.C. -> (none); device Inktime Library:NORDIC_NRF_3_CAPACITOR_0201_L -> Inktime Library:NORDIC_NRF_2_INDUCTOR_0402_L
- U$8: device Inktime Library:NORDIC_NRF_3_CAPACITOR_0201_L -> Inktime Library:NORDIC_NRF_2_INDUCTOR_0402_L
- renumbered U$10 to C18, U$12 to X1, U$15 to C19
Connections:
- removed net D+: D4.I/O2_2, U$29.D+@AD6
- removed net D-: D4.I/O1_2, U$29.D-@AD4
- removed net N$6: L3.1, L4.2
- new net D_N: D4.I/O1_2, U$31.D-@AD4
- new net D_P: D4.I/O2_2, U$31.D+@AD6
- new net N$3: U$4.1, U$8.2
- net 3V1: now also C35.1, U$31.DEC3V3@AC5; no longer U$27.2, U$29.DEC3V3@AC5
- net 3V3: now also C12.1, C13.1, C15.1, C22.1, C26.1, C3.1, C33.1, C36.1, U$31.VDD@A22, U$31.VDD@AD14, U$31.VDD@AD23, U$31.VDD@B1, U$31.VDD@W1, U$31.VDDH@Y2; no longer U$11.2, U$14.2, U$26.2, U$28.2, U$29.VDD@A22, U$29.VDD@AD14, U$29.VDD@AD23, U$29.VDD@B1, U$29.VDD@W1, U$29.VDDH@Y2, U$31.1, U$32.2, U$8.1, U$9.1
- net ALERT: now also U$31.P0.10/NFC2@J24; no longer U$29.P0.10/NFC2@J24
- net ANT: now also C29.1, U$31.ANT@H23, U$5.1; no longer L5.1, U$23.2, U$29.ANT@H23
- net DEC1: now also C30.1, U$31.DEC1@C1; no longer U$13.2, U$29.DEC1@C1
- net DEC3: now also C23.1, U$31.DEC3@D23; no longer U$16.2, U$29.DEC3@D23
- net DEC4_6: now also C14.1, C20.1, C24.1, U$31.DEC4@B5, U$31.DEC6@E24; no longer L3.2, U$17.2, U$29.DEC4@B5, U$29.DEC6@E24, U$5.2
- net EPD_3V3: now also C17.1, C48.2, L4.2; no longer L1.1, U$1.1, U$35.1
- net EPD_BUSY: now also U$31.P0.17@AD12; no longer U$29.P0.17@AD12
- net EPD_CS: now also U$31.P0.05/AIN3@K2; no longer U$29.P0.05/AIN3@K2
- net EPD_DC: now also U$31.P0.15@AD10; no longer U$29.P0.15@AD10
- net EPD_RST: now also U$31.P0.16@AC11; no longer U$29.P0.16@AC11
- net GND: now also C11.2, C12.2, C13.2, C14.2, C15.2, C17.2, C20.2, C21.2, C22.2, C23.2, C24.2, C25.2, C26.2, C27.2, C28.2, C29.2, C30.2, C31.2, C32.2, C33.2, C34.2, C35.2, C36.2, C37.1, C38.1, C39.1, C40.1, C41.1, C42.1, C43.1, C44.1, C45.1, C46.1, C47.1, C48.1, C49.2, U$22.2, U$22.4, U$31.VSS@B7, U$31.VSS_PA@F23, U$31.VSS_PAD; no longer U$1.2, U$11.1, U$13.1, U$14.1, U$16.1, U$17.1, U$18.2, U$19.1, U$20.4, U$21.1, U$22.1, U$23.1, U$24.1, U$25.1, U$26.1, U$27.1, U$28.1, U$29.VSS@B7, U$29.VSS_PA@F23, U$29.VSS_PAD, U$3.1, U$30.1, U$31.2, U$32.1, U$33.2, U$34.2, U$35.2, U$36.2, U$37.2, U$38.2, U$39.2, U$4.1, U$40.2, U$41.2, U$42.2, U$43.2, U$5.1, U$6.2, U$7.1, U$8.2, U$9.2
- net HAPTIC_EN: now also U$31.P0.12@U1; no longer U$29.P0.12@U1
- net IMU_INT1: now also U$31.P0.08@N1; no longer U$29.P0.08@N1
- net IMU_INT2: now also U$31.P1.08@P2; no longer U$29.P1.08@P2
- net MOSI: now also U$31.P0.03/AIN1@B13; no longer U$29.P0.03/AIN1@B13
- net N$1: now also U$31.P0.00/XL1@D2; no longer U$29.P0.00/XL1@D2
- net N$10: now also C31.1, C32.1, U$5.2; no longer L5.2, U$24.2, U$25.2
- net N$11: now also C21.1, U$31.DEC2@A18; no longer U$29.DEC2@A18, U$7.2
- net N$2: now also U$31.P0.01/XL2@F2; no longer U$29.P0.01/XL2@F2
- net N$20: now also C38.2; no longer U$33.1
- net N$21: now also C39.2; no longer U$34.1
- net N$23: now also C16.1; no longer U$2.1
- net N$25: now also C16.2, L4.1; no longer L1.2, U$2.2
- net N$31: now also C40.2; no longer U$36.1
- net N$32: now also C41.2; no longer U$37.1
- net N$33: now also C42.2; no longer U$38.1
- net N$34: now also C43.2; no longer U$39.1
- net N$36: now also C45.2; no longer U$41.1
- net N$38: now also C47.2; no longer U$43.1
- net N$5: now also U$31.DCC@B3, U$8.1; no longer L4.1, U$29.DCC@B3
- net N$8: now also C25.1, U$31.DEC5@N24; no longer U$22.2, U$29.DEC5@N24
- net P0.04: now also U$31.P0.04/AIN2@J1; no longer U$29.P0.04/AIN2@J1
- net P0.09: now also U$31.P0.09/NFC1@L24; no longer U$29.P0.09/NFC1@L24
- net P0.13: now also U$31.P0.13@AD8; no longer U$29.P0.13@AD8
- net P0.14: now also U$31.P0.14@AC9; no longer U$29.P0.14@AC9
- net P0.19: now also U$31.P0.19@AC15; no longer U$29.P0.19@AC15
- net P0.20: now also U$31.P0.20@AD16; no longer U$29.P0.20@AD16
- net P0.21: now also U$31.P0.21@AC17; no longer U$29.P0.21@AC17
- net P0.22: now also U$31.P0.22@AD18; no longer U$29.P0.22@AD18
- net P0.23: now also U$31.P0.23@AC19; no longer U$29.P0.23@AC19
- net P0.24: now also U$31.P0.24@AD20; no longer U$29.P0.24@AD20
- net P0.25: now also U$31.P0.25@AC21; no longer U$29.P0.25@AC21
- net P0.26: now also U$31.P0.26@G1; no longer U$29.P0.26@G1
- net P0.27: now also U$31.P0.27@H2; no longer U$29.P0.27@H2
- net P0.28: now also U$31.P0.28/AIN4@B11; no longer U$29.P0.28/AIN4@B11
- net P0.29: now also U$31.P0.29/AIN5@A10; no longer U$29.P0.29/AIN5@A10
- net P0.30: now also U$31.P0.30/AIN6@B9; no longer U$29.P0.30/AIN6@B9
- net P0.31: now also U$31.P0.31/AIN7@A8; no longer U$29.P0.31/AIN7@A8
- net P1.01: now also U$31.P1.01@Y23; no longer U$29.P1.01@Y23
- net P1.02: now also U$31.P1.02@W24; no longer U$29.P1.02@W24
- net P1.03: now also U$31.P1.03@V23; no longer U$29.P1.03@V23
- net P1.04: now also U$31.P1.04@U24; no longer U$29.P1.04@U24
- net P1.05: now also U$31.P1.05@T23; no longer U$29.P1.05@T23
- net P1.06: now also U$31.P1.06@R24; no longer U$29.P1.06@R24
- net P1.07: now also U$31.P1.07@P23; no longer U$29.P1.07@P23
- net P1.09: now also U$31.P1.09@R1; no longer U$29.P1.09@R1
- net P1.10: now also U$31.P1.10@A20; no longer U$29.P1.10@A20
- net P1.11: now also U$31.P1.11@B19; no longer U$29.P1.11@B19
- net P1.12: now also U$31.P1.12@B17; no longer U$29.P1.12@B17
- net P1.13: now also U$31.P1.13@A16; no longer U$29.P1.13@A16
- net P1.14: now also U$31.P1.14@B15; no longer U$29.P1.14@B15
- net P1.15: now also U$31.P1.15@A14; no longer U$29.P1.15@A14
- net PMIC_INT: now also U$31.P0.11@T2; no longer U$29.P0.11@T2
- net PREVGH: now also C44.2; no longer U$40.1
- net PREVGL: now also C46.2; no longer U$42.1
- net RESET: now also U$31.P0.18/RESET@AC13; no longer U$29.P0.18/RESET@AC13
- net SCK: now also U$31.P0.02/AIN0@A12; no longer U$29.P0.02/AIN0@A12
- net SCL: now also U$31.P0.07@M2; no longer U$29.P0.07@M2
- net SDA: now also U$31.P0.06@L1; no longer U$29.P0.06@L1
- net SWDCLK: now also U$31.SWDCLK@AA24; no longer U$29.SWDCLK@AA24
- net SWDIO: now also U$31.SWDIO@AC24; no longer U$29.SWDIO@AC24
- net SWO: now also U$31.P1.00@AD22; no longer U$29.P1.00@AD22
- net VBUS: now also C34.1, U$20.1, U$31.VBUS@AD2; no longer U$18.1, U$29.VBUS@AD2, U$30.2
- net VREG: now also C11.1, C37.2, C49.1; no longer C3.1, U$3.2, U$6.1
- net XC1: now also C28.1, U$22.1, U$31.XC1@B24; no longer U$20.1, U$21.2, U$29.XC1@B24
- net XC2: now also C27.1, U$22.3, U$31.XC2@A23; no longer U$19.2, U$20.3, U$29.XC2@A23
Other:
- moved on the sheet: C8, C9, D3, TP12, TP13
